File: ALAN_Carrier_board/carrier_board.brd (EAGLE design)
At the start: 124.7 x 100.8 mm, 38 parts, among them J1 POWER_JACKPTH, U1 LM317

Commit message: Gitignore and latest files
Parts:
- removed ENC_L, ENC_R: (no value), con-molex:KK-156-4
- added DC-POWER_OUT: (no value), pinhead:1X08
- added ENC_LEFT, ENC_RIGHT: (no value), pinhead:1X04/90
- moved USL 7.18 mm to (124.2, 61.0)
- moved USC 7.18 mm to (124.2, 94.2)
- moved USR 7.18 mm to (124.2, 77.5)
- moved ENC_NANO_R_OUT 0.36 mm to (57.9, 8.13)
- moved DC-COMMS 0.25 mm to (57.4, 70.6)
- moved US_NANO_R 0.06 mm to (112.1, 80.3)
- moved US_NANO_L 0.06 mm to (96.8, 80.3)
- turned US_NANO_R_OUT to 180 degrees
Connections:
- removed net DC-PWM14: DC-PWM.1
- removed net N$25: GPIO_D22-D53.2
- new net N$52: DC-POWER_OUT.2, POWER.7
- new net N$53: DC-POWER_OUT.3, POWER.6
- new net N$54: DC-POWER_OUT.4, POWER.5
- new net N$55: DC-POWER_OUT.5, POWER.4
- new net N$56: DC-POWER_OUT.6, POWER.3
- new net N$57: DC-POWER_OUT.7, POWER.2
- net DC-D22: now also GPIO_D22-D53.4; no longer GPIO_D22-D53.3
- net DC-D23: now also GPIO_D22-D53.3; no longer GPIO_D22-D53.4
- net DC-D24: now also GPIO_D22-D53.6; no longer GPIO_D22-D53.5
- net DC-D25: now also GPIO_D22-D53.5; no longer GPIO_D22-D53.6
- net DC-D26: now also GPIO_D22-D53.8; no longer GPIO_D22-D53.7
- net DC-D27: now also GPIO_D22-D53.7; no longer GPIO_D22-D53.8
- net DC-D28: now also GPIO_D22-D53.10; no longer GPIO_D22-D53.9
- net DC-D29: now also GPIO_D22-D53.9; no longer GPIO_D22-D53.10
- net DC-D30: now also GPIO_D22-D53.12; no longer GPIO_D22-D53.11
- net DC-D31: now also GPIO_D22-D53.11; no longer GPIO_D22-D53.12
- net DC-D32: now also GPIO_D22-D53.14; no longer GPIO_D22-D53.13
- net DC-D33: now also GPIO_D22-D53.13; no longer GPIO_D22-D53.14
- net DC-D34: now also GPIO_D22-D53.16; no longer GPIO_D22-D53.15
- net DC-D35: now also GPIO_D22-D53.15; no longer GPIO_D22-D53.16
- net DC-D36: now also GPIO_D22-D53.18; no longer GPIO_D22-D53.17
- net DC-D37: now also GPIO_D22-D53.17; no longer GPIO_D22-D53.18
- net DC-D38: now also GPIO_D22-D53.20; no longer GPIO_D22-D53.19
- net DC-D39: now also GPIO_D22-D53.19; no longer GPIO_D22-D53.20
- net DC-D40: now also GPIO_D22-D53.22; no longer GPIO_D22-D53.21
- net DC-D41: now also GPIO_D22-D53.21; no longer GPIO_D22-D53.22
- net DC-D42: now also GPIO_D22-D53.24; no longer GPIO_D22-D53.23
- net DC-D43: now also GPIO_D22-D53.23; no longer GPIO_D22-D53.24
- net DC-D44: now also GPIO_D22-D53.26; no longer GPIO_D22-D53.25
- net DC-D45: now also GPIO_D22-D53.25; no longer GPIO_D22-D53.26
- net DC-D46: now also GPIO_D22-D53.28; no longer GPIO_D22-D53.27
- net DC-D47: now also GPIO_D22-D53.27; no longer GPIO_D22-D53.28
- net DC-D48: now also GPIO_D22-D53.30; no longer GPIO_D22-D53.29
- net DC-D49: now also GPIO_D22-D53.29; no longer GPIO_D22-D53.30
- net DC-D50: now also GPIO_D22-D53.32; no longer GPIO_D22-D53.31
- net DC-D51: now also GPIO_D22-D53.31; no longer GPIO_D22-D53.32
- net DC-D52: now also GPIO_D22-D53.34; no longer GPIO_D22-D53.33
- net DC-D53: now also GPIO_D22-D53.33; no longer GPIO_D22-D53.34
- net DC-PWM13: now also DC-PWM.1
- net ENC_LA: now also ENC_LEFT.3; no longer ENC_L.3
- net ENC_LB: now also ENC_LEFT.4; no longer ENC_L.4
- net ENC_RA: now also ENC_RIGHT.3; no longer ENC_R.3
- net ENC_RB: now also ENC_RIGHT.4; no longer ENC_R.4
- net GND: now also ENC_LEFT.1, ENC_RIGHT.1; no longer ENC_L.1, ENC_R.1
- net N$6: now also GPIO_D22-D53_OUT.2
- net N$7: now also GPIO_D22-D53.2
- net N$9: now also DC-POWER_OUT.1, POWER.8; no longer GPIO_D22-D53_OUT.2
- net VCC: now also DC-POWER_OUT.8, ENC_LEFT.2, ENC_RIGHT.2, POWER.1; no longer ENC_L.2, ENC_R.2, POWER.8
Routing:
- net N$41: track 102.5 -> 54.3 mm
- net ENC_LA: track 120.6 -> 73.3 mm
- net N$40: track 95.2 -> 52.5 mm
- net N$42: track 89.0 -> 47.8 mm, vias 1 -> 0
- net N$13: track 111.5 -> 73.8 mm
- net DC-PWM13: track 0.00 -> 33.9 mm
- net GND: track 412.5 -> 444.7 mm, vias 2 -> 1
- net N$34: track 54.2 -> 81.4 mm, vias 2 -> 0
- net N$11: track 103.1 -> 78.6 mm, vias 1 -> 0
- net SDA: track 239.3 -> 262.9 mm, vias 3 -> 0
- net N$51: track 38.1 -> 59.4 mm, vias 1 -> 5
- net N$36: track 92.2 -> 71.0 mm
- net N$33: track 67.6 -> 85.0 mm
- net 1INA: track 100.7 -> 84.5 mm
- net N$38: track 102.4 -> 86.7 mm, vias 1 -> 0
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Other:
- outline, holes or cut-outs redrawn
- board text added: "1INA"
- board text added: "1INB"
- board text added: "1PWM"
- board text added: "2INA"
- board text added: "2INB"
- board text added: "2PWM"
- board text added: "Arduino Mega 2560 Drive Controller"
- board text added: "D10"
- board text added: "D11"
- board text added: "D12"
- board text added: "D13"
- board text added: "D22"
- board text added: "D4"
- board text added: "D53"
- board text added: "D6"
- board text added: "DC Comms"
- board text added: "DC PWM"
- board text added: "Drive Controller Power/Analog"
- board text added: "ENC LEFT"
- board text added: "ENC RIGHT"
- board text added: "Encoder Nano"
- board text added: "Power Supply"
- board text added: "RX0"
- board text added: "RX1"
- board text added: "RX2"
- board text added: "RX3"
- board text added: "SCL"
- board text added: "SCL1"
- board text added: "SDA"
- board text added: "SDA1"
- board text added: "TX0"
- board text added: "TX1"
- board text added: "TX2"
- board text added: "TX3"
- board text added: "US CENTER"
- board text added: "US LEFT"
- board text added: "US RIGHT"
- board text added: "Ultrasonic Nano"
