File: ALAN_Carrier_board/carrier_board.sch (EAGLE design)
At the start: 38 parts, among them J1 POWER_JACKPTH, U1 LM317

Commit message: Gitignore and latest files
Parts:
- removed ENC_L, ENC_R: (no value), con-molex:KK-156-4
- added DC-POWER_OUT: (no value), pinhead:PINHD-1X8
- added ENC_LEFT, ENC_RIGHT: (no value), pinhead:PINHD-1X4/90
Connections:
- removed net DC-PWM14: DC-PWM.1
- removed net N$25: GPIO_D22-D53.2
- new net N$52: DC-POWER_OUT.2, POWER.7
- new net N$53: DC-POWER_OUT.3, POWER.6
- new net N$54: DC-POWER_OUT.4, POWER.5
- new net N$55: DC-POWER_OUT.5, POWER.4
- new net N$56: DC-POWER_OUT.6, POWER.3
- new net N$57: DC-POWER_OUT.7, POWER.2
- net DC-D22: now also GPIO_D22-D53.4; no longer GPIO_D22-D53.3
- net DC-D23: now also GPIO_D22-D53.3; no longer GPIO_D22-D53.4
- net DC-D24: now also GPIO_D22-D53.6; no longer GPIO_D22-D53.5
- net DC-D25: now also GPIO_D22-D53.5; no longer GPIO_D22-D53.6
- net DC-D26: now also GPIO_D22-D53.8; no longer GPIO_D22-D53.7
- net DC-D27: now also GPIO_D22-D53.7; no longer GPIO_D22-D53.8
- net DC-D28: now also GPIO_D22-D53.10; no longer GPIO_D22-D53.9
- net DC-D29: now also GPIO_D22-D53.9; no longer GPIO_D22-D53.10
- net DC-D30: now also GPIO_D22-D53.12; no longer GPIO_D22-D53.11
- net DC-D31: now also GPIO_D22-D53.11; no longer GPIO_D22-D53.12
- net DC-D32: now also GPIO_D22-D53.14; no longer GPIO_D22-D53.13
- net DC-D33: now also GPIO_D22-D53.13; no longer GPIO_D22-D53.14
- net DC-D34: now also GPIO_D22-D53.16; no longer GPIO_D22-D53.15
- net DC-D35: now also GPIO_D22-D53.15; no longer GPIO_D22-D53.16
- net DC-D36: now also GPIO_D22-D53.18; no longer GPIO_D22-D53.17
- net DC-D37: now also GPIO_D22-D53.17; no longer GPIO_D22-D53.18
- net DC-D38: now also GPIO_D22-D53.20; no longer GPIO_D22-D53.19
- net DC-D39: now also GPIO_D22-D53.19; no longer GPIO_D22-D53.20
- net DC-D40: now also GPIO_D22-D53.22; no longer GPIO_D22-D53.21
- net DC-D41: now also GPIO_D22-D53.21; no longer GPIO_D22-D53.22
- net DC-D42: now also GPIO_D22-D53.24; no longer GPIO_D22-D53.23
- net DC-D43: now also GPIO_D22-D53.23; no longer GPIO_D22-D53.24
- net DC-D44: now also GPIO_D22-D53.26; no longer GPIO_D22-D53.25
- net DC-D45: now also GPIO_D22-D53.25; no longer GPIO_D22-D53.26
- net DC-D46: now also GPIO_D22-D53.28; no longer GPIO_D22-D53.27
- net DC-D47: now also GPIO_D22-D53.27; no longer GPIO_D22-D53.28
- net DC-D48: now also GPIO_D22-D53.30; no longer GPIO_D22-D53.29
- net DC-D49: now also GPIO_D22-D53.29; no longer GPIO_D22-D53.30
- net DC-D50: now also GPIO_D22-D53.32; no longer GPIO_D22-D53.31
- net DC-D51: now also GPIO_D22-D53.31; no longer GPIO_D22-D53.32
- net DC-D52: now also GPIO_D22-D53.34; no longer GPIO_D22-D53.33
- net DC-D53: now also GPIO_D22-D53.33; no longer GPIO_D22-D53.34
- net DC-PWM13: now also DC-PWM.1
- net ENC_LA: now also ENC_LEFT.3; no longer ENC_L-3.S
- net ENC_LB: now also ENC_LEFT.4; no longer ENC_L-4.S
- net ENC_RA: now also ENC_RIGHT.3; no longer ENC_R-3.S
- net ENC_RB: now also ENC_RIGHT.4; no longer ENC_R-4.S
- net GND: now also ENC_LEFT.1, ENC_RIGHT.1; no longer ENC_L-1.S, ENC_R-1.S
- net N$6: now also GPIO_D22-D53_OUT.2
- net N$7: now also GPIO_D22-D53.2
- net N$9: now also DC-POWER_OUT.1, POWER.8; no longer GPIO_D22-D53_OUT.2
- net VCC: now also DC-POWER_OUT.8, ENC_LEFT.2, ENC_RIGHT.2, POWER.1; no longer ENC_L-2.S, ENC_R-2.S, POWER.8
